File: pcb/startrckr_pcb.kicad_pcb (KiCad board)
At the start: 2 copper layers, 76.2 x 69.9 mm, 59 parts, among them J1 USB_B, J10 M3, J2 M1, J3 Micro_SD_Card, J4 12V, J5 USB_BOOT, J6 LS1, J7 LS2, J8 LS3, J9 M2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

Commit message: clean up + power jack
Parts:
- removed C1: 10u, Capacitor_SMD:C_0603_1608Metric_Pad1.08x0.95mm_HandSolder
- removed J3: Micro_SD_Card, Connector_Card:microSD_HC_Wuerth_693072010801
- added J11: Barrel_Jack_Switch, Connector_BarrelJack:BarrelJack_Horizontal, F.Cu at (228.0, 67.6)
- added U4: BNO055, Package_LGA:LGA-28_5.2x3.8mm_P0.5mm, F.Cu at (136.9, 76.1)
- R11: value R -> 1k
- moved G*** 54.0 mm to (132.7, 97.2)
- moved J4 24.3 mm to (240.7, 41.9)
Routing:
- net SD_CS: track 49.8 -> 0.00 mm
- net SD_MOSI: track 47.9 -> 0.00 mm
- net SD_MISO: track 46.7 -> 0.00 mm, vias 2 -> 0
- net SD_CLK: track 46.3 -> 0.00 mm
- net +3V3: track 105.3 -> 88.5 mm
- net GND: track 8.58 -> 6.82 mm, vias 14 -> 13

Commit message: Schematic update
Parts:
- removed J4: 12V, TerminalBlock:TerminalBlock_bornier-2_P5.08mm
- removed U4: BNO055, Package_LGA:LGA-28_5.2x3.8mm_P0.5mm
- added J12: SPI1, Connector_Molex:Molex_KK-254_AE-6410-06A_1x06_P2.54mm_Vertical, F.Cu at (120.0, 64.5)
- added J13: SPI2, Connector_Molex:Molex_KK-254_AE-6410-06A_1x06_P2.54mm_Vertical, F.Cu at (120.0, 72.4)
- added J14: UART, Connector_Molex:Molex_KK-254_AE-6410-04A_1x04_P2.54mm_Vertical, F.Cu at (107.8, 46.8)
- added J15: I2C1, Connector_Molex:Molex_KK-254_AE-6410-04A_1x04_P2.54mm_Vertical, F.Cu at (107.8, 54.6)
- added J16: I2C1, Connector_Molex:Molex_KK-254_AE-6410-04A_1x04_P2.54mm_Vertical, F.Cu at (107.8, 62.5)
- added J17: I2C2, Connector_Molex:Molex_KK-254_AE-6410-05A_1x05_P2.54mm_Vertical, F.Cu at (128.7, 54.6)
- added J3: I2C2, Connector_Molex:Molex_KK-254_AE-6410-05A_1x05_P2.54mm_Vertical, F.Cu at (128.7, 46.8)
- added JP11: J_SPI_3V3, Jumper:SolderJumper-2_P1.3mm_Open_Pad1.0x1.5mm, F.Cu at (119.9, 44.6)
- added JP12: J_SPI_5V, Jumper:SolderJumper-2_P1.3mm_Open_Pad1.0x1.5mm, F.Cu at (119.9, 48.2)
- added JP13: J_SPI_3V3, Jumper:SolderJumper-2_P1.3mm_Open_Pad1.0x1.5mm, F.Cu at (119.9, 51.7)
- added JP14: J_SPI_5V, Jumper:SolderJumper-2_P1.3mm_Open_Pad1.0x1.5mm, F.Cu at (119.9, 55.3)
- added JP15: J_SPI_3V3, Jumper:SolderJumper-2_P1.3mm_Open_Pad1.0x1.5mm, F.Cu at (119.9, 58.8)
- added JP16: J_SPI_5V, Jumper:SolderJumper-2_P1.3mm_Open_Pad1.0x1.5mm, F.Cu at (124.2, 44.6)
- added JP17: J_SPI_3V3, Jumper:SolderJumper-2_P1.3mm_Open_Pad1.0x1.5mm, F.Cu at (124.2, 48.2)
- added JP18: J_SPI_5V, Jumper:SolderJumper-2_P1.3mm_Open_Pad1.0x1.5mm, F.Cu at (124.2, 51.7)
- added JP19: J_SPI_3V3, Jumper:SolderJumper-2_P1.3mm_Open_Pad1.0x1.5mm, F.Cu at (124.2, 55.3)
- added JP20: J_SPI_5V, Jumper:SolderJumper-2_P1.3mm_Open_Pad1.0x1.5mm, F.Cu at (124.2, 58.8)
- J6, J7, J8: footprint Connector_PinSocket_2.54mm:PinSocket_1x02_P2.54mm_Vertical -> Connector_Molex:Molex_KK-254_AE-6410-02A_1x02_P2.54mm_Vertical
- moved G*** 83.2 mm to (194.9, 32.4)
- moved J6 70.1 mm to (115.6, 137.8)
- moved J7 67.2 mm to (122.6, 137.8)
- moved J8 64.4 mm to (129.5, 137.8)
- moved JP4 36.6 mm to (136.0, 113.1)
- moved BZ1 36.6 mm to (132.1, 116.8)
- moved R7 36.6 mm to (136.1, 108.8)
- moved J11 29.2 mm to (198.8, 68.6)
- moved D1 21.9 mm to (141.4, 97.3)
- moved D2 21.9 mm to (141.4, 101.3)
- moved D3 21.9 mm to (141.4, 105.3)
- moved R4 21.9 mm to (146.4, 97.3)
- moved R5 21.9 mm to (146.4, 101.4)
- moved R6 21.9 mm to (146.4, 105.4)
- moved C12 18.6 mm to (180.0, 120.7)
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Connections:
- U1 pad 13: unconnected-(U1-GPIO10-Pad13) -> I2C1_SDA
- U1 pad 14: unconnected-(U1-GPIO11-Pad14) -> I2C1_SCL
- U1 pad 18: unconnected-(U1-GPIO15-Pad18) -> SPI_CS2
- U1 pad 2: unconnected-(U1-GPIO0-Pad2) -> UART_TX
- U1 pad 3: unconnected-(U1-GPIO1-Pad3) -> UART_RX
- U1 pad 38: unconnected-(U1-GPIO26_ADC0-Pad38) -> I2C2_SDA
- U1 pad 39: unconnected-(U1-GPIO27_ADC1-Pad39) -> I2C2_SCL
- U1 pad 4: SD_CLK -> SPI_CLK
- U1 pad 40: unconnected-(U1-GPIO28_ADC2-Pad40) -> I2C2_DRDY
- U1 pad 5: SD_MOSI -> SPI_MOSI
- U1 pad 6: SD_MISO -> SPI_MISO
- U1 pad 7: SD_CS -> SPI_CS1
Routing:
- net +3V3: track 88.5 -> 52.7 mm, vias 4 -> 1
- net M3_DIR: track 33.1 -> 0.00 mm
- net +1V1: track 34.2 -> 2.99 mm, vias 4 -> 0
- net M3_STEP: track 30.5 -> 0.00 mm
- net M1_STEP: track 32.5 -> 5.40 mm
- net M1_ENABLE: track 47.8 -> 21.2 mm
- net M1_DIR: track 30.5 -> 4.84 mm
- net LS3: track 22.3 -> 0.00 mm
- net M2_ENABLE: track 25.9 -> 3.90 mm
- net LED3: track 20.6 -> 0.00 mm
- net M3_ENABLE: track 19.3 -> 0.00 mm
- net LS2: track 18.9 -> 0.00 mm
- net LED2: track 18.3 -> 0.00 mm
- net USB_DM: track 18.5 -> 0.62 mm, vias 1 -> 0
- net LS1: track 17.3 -> 0.00 mm
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Other:
- board size 76.2 x 69.9 mm -> 73.4 x 100.3 mm
- board text added: "StarTrckr V2"
- board text removed: "+ PWR -"
- board text removed: "StarTrckr V1"

Commit message: PCB V2 ready
Parts:
- removed the G*** at (132.7, 97.2)
- added TP_12V1: TP, TestPoint:TestPoint_Pad_D1.5mm, F.Cu at (202.1, 74.3)
- added TP_3V3: TP, TestPoint:TestPoint_Pad_D1.5mm, F.Cu at (192.4, 82.5)
- added TP_5V1: TP, TestPoint:TestPoint_Pad_D1.5mm, F.Cu at (197.5, 74.3)
- G***, JP11, JP12, JP13, JP14, JP15, JP16, JP17, JP18, JP19, JP20: moved to B.Cu
- I2C1_1: renamed from J16; footprint Connector_Molex:Molex_KK-254_AE-6410-04A_1x04_P2.54mm_Vertical -> Connector_JST:JST_XH_B4B-XH-A_1x04_P2.50mm_Vertical
- I2C1_2: renamed from J15; footprint Connector_Molex:Molex_KK-254_AE-6410-04A_1x04_P2.54mm_Vertical -> Connector_JST:JST_XH_B4B-XH-A_1x04_P2.50mm_Vertical
- I2C2_1: renamed from J3; footprint Connector_Molex:Molex_KK-254_AE-6410-05A_1x05_P2.54mm_Vertical -> Connector_JST:JST_XH_B5B-XH-A_1x05_P2.50mm_Vertical
- I2C2_2: renamed from J17; footprint Connector_Molex:Molex_KK-254_AE-6410-05A_1x05_P2.54mm_Vertical -> Connector_JST:JST_XH_B5B-XH-A_1x05_P2.50mm_Vertical
- J5: value USB_BOOT -> BOOT
- LS1: renamed from J6; footprint Connector_Molex:Molex_KK-254_AE-6410-02A_1x02_P2.54mm_Vertical -> Connector_JST:JST_XH_B2B-XH-A_1x02_P2.50mm_Vertical
- LS2: renamed from J7; footprint Connector_Molex:Molex_KK-254_AE-6410-02A_1x02_P2.54mm_Vertical -> Connector_JST:JST_XH_B2B-XH-A_1x02_P2.50mm_Vertical
- LS3: renamed from J8; footprint Connector_Molex:Molex_KK-254_AE-6410-02A_1x02_P2.54mm_Vertical -> Connector_JST:JST_XH_B2B-XH-A_1x02_P2.50mm_Vertical
- SPI1: renamed from J12; footprint Connector_Molex:Molex_KK-254_AE-6410-06A_1x06_P2.54mm_Vertical -> Connector_JST:JST_XH_B6B-XH-A_1x06_P2.50mm_Vertical
- SPI2: renamed from J13; footprint Connector_Molex:Molex_KK-254_AE-6410-06A_1x06_P2.54mm_Vertical -> Connector_JST:JST_XH_B6B-XH-A_1x06_P2.50mm_Vertical
- UART1: renamed from J14; footprint Connector_Molex:Molex_KK-254_AE-6410-04A_1x04_P2.54mm_Vertical -> Connector_JST:JST_XH_B4B-XH-A_1x04_P2.50mm_Vertical
- moved I2C2_1 96.9 mm to (200.7, 111.8), turned to -90 degrees
- moved I2C1_1 96.9 mm to (182.2, 124.6), turned to -90 degrees
- moved JP16 96.9 mm to (198.1, 107.3), turned to 90 degrees
- moved I2C1_2 96.7 mm to (174.6, 124.6), turned to -90 degrees
- moved JP15 94.8 mm to (201.3, 107.3), turned to 90 degrees
- moved I2C2_2 86.5 mm to (193.6, 111.8), turned to -90 degrees
- moved BZ1 84.7 mm to (214.9, 134.9)
- moved JP11 84.7 mm to (184.8, 99.1), turned to 90 degrees
- moved JP19 84.6 mm to (177.2, 121.3), turned to 90 degrees
- moved JP20 83.5 mm to (179.7, 121.3), turned to 90 degrees
- moved UART1 82.0 mm to (174.0, 95.3)
- moved JP12 80.5 mm to (182.2, 99.1), turned to 90 degrees
- moved JP4 79.9 mm to (214.0, 130.2), turned to -90 degrees
- moved R7 77.7 mm to (210.8, 130.2), turned to 90 degrees
- moved LS3 75.8 mm to (205.1, 131.4), turned to -90 degrees
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Routing:
- net +3V3: track 52.7 -> 164.9 mm, vias 1 -> 4
- net +5V: track 115.7 -> 226.9 mm, vias 0 -> 6
- net I2C1_SCL: track 0.00 -> 54.7 mm
- net I2C1_SDA: track 0.00 -> 47.2 mm
- net I2C2_DRDY: track 0.00 -> 46.4 mm, vias 0 -> 1
- net BUZZER: track 4.43 -> 49.3 mm, vias 1 -> 3
- net LS3: track 0.00 -> 43.2 mm
- net SPI_CS1: track 0.00 -> 41.8 mm
- net I2C2_SCL: track 0.00 -> 39.7 mm, vias 0 -> 1
- net I2C2_SDA: track 0.00 -> 38.8 mm, vias 0 -> 2
- net LS2: track 0.00 -> 37.6 mm
- net SPI_MISO: track 0.00 -> 36.5 mm
- net LS1: track 0.00 -> 34.7 mm
- net SPI_MOSI: track 0.00 -> 34.4 mm
- net M3_DIR: track 0.00 -> 33.0 mm
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Other:
- board size 73.4 x 100.3 mm -> 60 x 85 mm
- board text added: "I2C1 3V3"
- board text added: "I2C1 5V"
- board text added: "I2C2 3V3"
- board text added: "I2C2 5V"
- board text added: "NIKODEM BARTNIK INDYSTRY.CC 18.03.2024"
- board text added: "SPI1 3V3"
- board text added: "SPI1 5V"
- board text added: "SPI2 3V3"
- board text added: "SPI2 5V"
- board text added: "UART 3V3"
- board text added: "UART 5V"
- board text removed: "NIKODEM BARTNIK INDYSTRY.CC 07.10.2022"
