File: pcb/startrckr_pcb.kicad_sch (KiCad schematic)
At the start: 57 parts, among them J1 USB_B, J10 M3, J2 M1, J3 Micro_SD_Card, J4 12V, J5 USB_BOOT, J6 LS1, J7 LS2, J8 LS3, J9 M2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

Commit message: values update
Parts:
- R11: value R -> 1k
Changed lines of the file:
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@@
-    )
-  )
-  (global_label "SD_CLK" (shape input) (at 234.95 125.73 0) (fields_autoplaced)
-    (effects (font (size 1.27 1.27)) (justify left))
-    (property "Intersheet References" "${INTERSHEET_REFS}" (id 0) (at 244.3783 125.8094 0)
-      (effects (font (size 1.27 1.27)) (justify left) hide)
     )
   )
@@
     (in_bom yes) (on_board yes) (fields_autoplaced)
     (property "Reference" "R11" (id 0) (at 177.8 251.46 90))
-    (property "Value" "R" (id 1) (at 177.8 254 90))
+    (property "Value" "1k" (id 1) (at 177.8 254 90))
     (property "Footprint" "Resistor_SMD:R_0603_1608Metric_Pad0.98x0.95mm_HandSolder" (id 2) (at 177.8 259.588 90)
       (effects (font (size 1.27 1.27)) hide)
@@
     )
     (path "/511ba78e-1c39-456e-9092-6fdf5076d120"
-      (reference "R11") (unit 1) (value "R") (footprint "Resistor_SMD:R_0603_1608Metric_Pad0.98x0.95mm_HandSolder")
+      (reference "R11") (unit 1) (value "1k") (footprint "Resistor_SMD:R_0603_1608Metric_Pad0.98x0.95mm_HandSolder")
     )
     (path "/3f7c9122-5391-41a7-b888-6a9ff16f7acc"

Commit message: clean up + power jack
Parts:
- removed C1: 10u, Capacitor_SMD:C_0603_1608Metric_Pad1.08x0.95mm_HandSolder, symbol Device:C
- removed J3: Micro_SD_Card, Connector_Card:microSD_HC_Wuerth_693072010801, symbol Connector:Micro_SD_Card
- added J11: Barrel_Jack_Switch, Connector_BarrelJack:BarrelJack_Horizontal, symbol Connector:Barrel_Jack_Switch
- added U4: BNO055, Package_LGA:LGA-28_5.2x3.8mm_P0.5mm, symbol Sensor_Motion:BNO055
Connections:
- net +12V: now also J11.1
- net GND: now also J11.2
- new net: U4.15 (GNDIO), U4.16 (GNDIO), U4.25 (GNDIO)
Other:
- note added: "IMU"
- note removed: "SD CARD"
- moved on the sheet: J4

Commit message: Schematic update
Parts:
- removed J4: 12V, TerminalBlock:TerminalBlock_bornier-2_P5.08mm, symbol Connector:Screw_Terminal_01x02
- removed U4: BNO055, Package_LGA:LGA-28_5.2x3.8mm_P0.5mm, symbol Sensor_Motion:BNO055
- added J12: SPI1, Connector_Molex:Molex_KK-254_AE-6410-06A_1x06_P2.54mm_Vertical, symbol Connector_Generic:Conn_01x06
- added J13: SPI2, Connector_Molex:Molex_KK-254_AE-6410-06A_1x06_P2.54mm_Vertical, symbol Connector_Generic:Conn_01x06
- added J14: UART, Connector_Molex:Molex_KK-254_AE-6410-04A_1x04_P2.54mm_Vertical, symbol Connector_Generic:Conn_01x04
- added J15, J16: I2C1, Connector_Molex:Molex_KK-254_AE-6410-04A_1x04_P2.54mm_Vertical, symbol Connector_Generic:Conn_01x04
- added J17, J3: I2C2, Connector_Molex:Molex_KK-254_AE-6410-05A_1x05_P2.54mm_Vertical, symbol Connector_Generic:Conn_01x05
- added JP11, JP13, JP15, JP17, JP19: J_SPI_3V3, Jumper:SolderJumper-2_P1.3mm_Open_Pad1.0x1.5mm, symbol Jumper:SolderJumper_2_Open
- added JP12, JP14, JP16, JP18, JP20: J_SPI_5V, Jumper:SolderJumper-2_P1.3mm_Open_Pad1.0x1.5mm, symbol Jumper:SolderJumper_2_Open
- J6, J7, J8: footprint Connector_PinSocket_2.54mm:PinSocket_1x02_P2.54mm_Vertical -> Connector_Molex:Molex_KK-254_AE-6410-02A_1x02_P2.54mm_Vertical
Connections:
- net +3V3: now also JP12.2 (B), JP14.2 (B), JP16.2 (B), JP18.2 (B), JP20.2 (B)
- net +5V: now also JP11.2 (B), JP13.2 (B), JP15.2 (B), JP17.2 (B), JP19.2 (B)
- net GND: now also J12.2 (Pin_2), J13.2 (Pin_2), J14.2 (Pin_2), J15.2 (Pin_2), J16.2 (Pin_2), J17.2 (Pin_2), J3.2 (Pin_2)
- net I2C1_SDA: now reaches U1.13 (GPIO10)
- net I2C1_SDA: now also J15.4 (Pin_4), J16.4 (Pin_4)
- net I2C1_SCL: now reaches U1.14 (GPIO11)
- net I2C1_SCL: now also J15.3 (Pin_3), J16.3 (Pin_3)
- net SPI_CS2: now reaches U1.18 (GPIO15)
- net SPI_CS2: now also J13.3 (Pin_3)
- net UART_TX: now reaches U1.2 (GPIO0)
- net UART_TX: now also J14.4 (Pin_4)
- net UART_RX: now reaches U1.3 (GPIO1)
- net UART_RX: now also J14.3 (Pin_3)
- net I2C2_SDA: now reaches U1.38 (GPIO26_ADC0)
- net I2C2_SDA: now also J17.4 (Pin_4), J3.4 (Pin_4)
- net I2C2_SCL: now reaches U1.39 (GPIO27_ADC1)
- net I2C2_SCL: now also J17.3 (Pin_3), J3.3 (Pin_3)
- net I2C2_DRDY: now reaches U1.40 (GPIO28_ADC2)
- net I2C2_DRDY: now also J17.5 (Pin_5), J3.5 (Pin_5)
- net SD_CLK renamed SPI_CLK
- net SPI_CLK: now also J12.4 (Pin_4), J13.4 (Pin_4)
- net SD_CS renamed SPI_CS1
- net SPI_CS1: now also J12.3 (Pin_3)
- net SD_MISO renamed SPI_MISO
- net SPI_MISO: now also J12.6 (Pin_6), J13.6 (Pin_6)
- net SD_MOSI renamed SPI_MOSI
- net SPI_MOSI: now also J12.5 (Pin_5), J13.5 (Pin_5)
- new net: J12.1 (Pin_1), JP11.1 (A), JP12.1 (A)
- new net: J17.1 (Pin_1), J3.1 (Pin_1), JP15.1 (A), JP16.1 (A)
- new net: J15.1 (Pin_1), J16.1 (Pin_1), JP19.1 (A), JP20.1 (A)
- new net: J14.1 (Pin_1), JP17.1 (A), JP18.1 (A)
- new net: J13.1 (Pin_1), JP13.1 (A), JP14.1 (A)
Other:
- note added: "CONNECTORS"
- note added: "STARTRCKR PCB V2"
- note removed: "IMU"
- note removed: "STARTRCKR PCB V1"
- moved on the sheet: BZ1, D1, D2, D3, J11, JP4, R4, R5, R6, R7

Commit message: PCB V2 ready
Parts:
- added TP_12V1, TP_3V3, TP_5V1: TP, TestPoint:TestPoint_Pad_D1.5mm, symbol Connector:TestPoint_Alt
- I2C1_1: renamed from J16; footprint Connector_Molex:Molex_KK-254_AE-6410-04A_1x04_P2.54mm_Vertical -> Connector_JST:JST_XH_B4B-XH-A_1x04_P2.50mm_Vertical
- I2C1_2: renamed from J15; footprint Connector_Molex:Molex_KK-254_AE-6410-04A_1x04_P2.54mm_Vertical -> Connector_JST:JST_XH_B4B-XH-A_1x04_P2.50mm_Vertical
- I2C2_1: renamed from J3; footprint Connector_Molex:Molex_KK-254_AE-6410-05A_1x05_P2.54mm_Vertical -> Connector_JST:JST_XH_B5B-XH-A_1x05_P2.50mm_Vertical
- I2C2_2: renamed from J17; footprint Connector_Molex:Molex_KK-254_AE-6410-05A_1x05_P2.54mm_Vertical -> Connector_JST:JST_XH_B5B-XH-A_1x05_P2.50mm_Vertical
- LS1: renamed from J6; footprint Connector_Molex:Molex_KK-254_AE-6410-02A_1x02_P2.54mm_Vertical -> Connector_JST:JST_XH_B2B-XH-A_1x02_P2.50mm_Vertical
- LS2: renamed from J7; footprint Connector_Molex:Molex_KK-254_AE-6410-02A_1x02_P2.54mm_Vertical -> Connector_JST:JST_XH_B2B-XH-A_1x02_P2.50mm_Vertical
- LS3: renamed from J8; footprint Connector_Molex:Molex_KK-254_AE-6410-02A_1x02_P2.54mm_Vertical -> Connector_JST:JST_XH_B2B-XH-A_1x02_P2.50mm_Vertical
- SPI1: renamed from J12; footprint Connector_Molex:Molex_KK-254_AE-6410-06A_1x06_P2.54mm_Vertical -> Connector_JST:JST_XH_B6B-XH-A_1x06_P2.50mm_Vertical
- SPI2: renamed from J13; footprint Connector_Molex:Molex_KK-254_AE-6410-06A_1x06_P2.54mm_Vertical -> Connector_JST:JST_XH_B6B-XH-A_1x06_P2.50mm_Vertical
- UART1: renamed from J14; footprint Connector_Molex:Molex_KK-254_AE-6410-04A_1x04_P2.54mm_Vertical -> Connector_JST:JST_XH_B4B-XH-A_1x04_P2.50mm_Vertical
Connections:
- net +12V: now also TP_12V1.1
- net +3V3: now also TP_3V3.1
- net +5V: now also TP_5V1.1
